Commit message: fix: use velocity controllers and tune wheel dynamics
- Switch wheel controllers from effort to velocity type
- Switch wheel transmission to VelocityJointInterface
- Add wheel friction 0.1, update velocity limit to 273 rad/s
- Disable rviz auto-launch from launch file

File: urdf/unicorn.urdf (robot description, URDF)
Before this commit: robot unicorn, 12 links, 11 joints
Joints:
- joint left_front_wheel_joint: limit effort=10 velocity=100 -> effort=10 velocity=273
- joint left_rear_wheel_joint: limit effort=10 velocity=100 -> effort=10 velocity=273
- joint right_front_wheel_joint: limit effort=10 velocity=100 -> effort=10 velocity=273
- joint right_rear_wheel_joint: limit effort=10 velocity=100 -> effort=10 velocity=273

Commit message: feat: add PID velocity control, increase wheel effort/friction, fix odom twist to body frame

File: urdf/unicorn.urdf (robot description, URDF)
Before this commit: robot unicorn, 12 links, 11 joints
Joints:
- joint left_front_wheel_joint: limit effort=10 velocity=273 -> effort=100 velocity=273
- joint left_rear_wheel_joint: limit effort=10 velocity=273 -> effort=100 velocity=273
- joint right_front_wheel_joint: limit effort=10 velocity=273 -> effort=100 velocity=273
- joint right_rear_wheel_joint: limit effort=10 velocity=273 -> effort=100 velocity=273

Commit message: feat: add L515 LiDAR camera simulation with distance-dependent depth noise
- Add realsense_gazebo_plugin and realsense2_description to thirdparty
- Create unicorn_l515.urdf (vehicle + L515 front-mounted)
- Create unicorn_l515_pitched.urdf (LiDAR pitched 15deg downward)
- Implement distance-dependent depth noise: stddev(d) = 0.004 + 0.00111*d
- Optimized point cloud generation with pre-computed LUT
- Replace Mid-360 mesh with STP-converted STL
- Update icra_racetrack.launch to use pitched variant with RViz

File: urdf/unicorn.urdf (robot description, URDF)
Before this commit: robot unicorn, 12 links, 11 joints
Links:
- link livox_mid360: geometry visual mesh filename=package://roboracer_gazebo/meshes/mid360.stl
