Commit message: feat: update vehicle specs to match real car dimensions
- Wheelbase: 325mm -> 360mm
- Front track: 200mm -> 302mm, Rear track: 200mm -> 296mm
- Chassis mass: 4.0kg -> 1.7kg, wheel mass: 0.34kg -> 0.12kg
- Wheel radius: 50mm -> 55mm, width: 45mm -> 26mm
- Max steering angle: ±57deg -> ±62deg (1.08 rad)
- Recalculated inertia tensors for all bodies
- Updated launch params and documentation

File: urdf/macros.xacro (robot description, xacro)
@@ -3,30 +3,33 @@
 <!-- inertial parameter macros -->
 <xacro:macro name="chassis_inertial_params">
-  <origin xyz="0.1477 0 0" rpy="0 0 0" />
-  <mass value="4.0" />
-  <inertia ixx="0.010609" ixy="0"          ixz="0"
-                          iyy="0.050409"   iyz="0"
-                                           izz="0.05865" />
+  <!-- CoG at ~half wheelbase forward from rear axle (base_link) -->
+  <origin xyz="0.18 0 0" rpy="0 0 0" />
+  <mass value="1.70" />
+  <!-- Box approx: 0.56 x 0.302 x 0.06, m=1.7 -->
+  <inertia ixx="0.01343" ixy="0"          ixz="0"
+                          iyy="0.04494"   iyz="0"
+                                           izz="0.05739" />
 </xacro:macro>
 <xacro:macro name="left_wheels_inertial_params">
-  <origin xyz="0 0 -0.0225" rpy="0 0 0" />
-  <mass value="0.34055" />
-  <inertia ixx="0.00026046" ixy="0"          ixz="0"
-                            iyy="0.00026046" iyz="0"
-                                             izz="0.00041226" />
+  <origin xyz="0 0 -0.013" rpy="0 0 0" />
+  <mass value="0.12" />
+  <!-- Cylinder: r=0.055, h=0.026, m=0.12 -->
+  <inertia ixx="0.0000975" ixy="0"          ixz="0"
+                            iyy="0.0000975" iyz="0"
+                                             izz="0.0001815" />
 </xacro:macro>
 <xacro:macro name="right_wheels_inertial_params">
-  <origin xyz="0 0 0.0225" rpy="0 0 0" />
-  <mass value="0.34055" />
-  <inertia ixx="0.00026046" ixy="0"          ixz="0"
-                            iyy="0.00026046" iyz="0"
-                                             izz="0.00041226" />
+  <origin xyz="0 0 0.013" rpy="0 0 0" />
+  <mass value="0.12" />
+  <inertia ixx="0.0000975" ixy="0"          ixz="0"
+                            iyy="0.0000975" iyz="0"
+                                             izz="0.0001815" />
 </xacro:macro>
 <xacro:macro name="steering_hinge_inertial_params">
   <origin xyz="0 0 0" rpy="0 0 0" />
-  <mass value="0.100" />
-  <inertia ixx="4E-06" ixy="0"           ixz="0"
-                            iyy="4E-06"  iyz="0"
-                                              izz="4E-06" />
+  <mass value="0.05" />
+  <inertia ixx="2E-06" ixy="0"           ixz="0"
+                            iyy="2E-06"  iyz="0"
+                                              izz="2E-06" />
 </xacro:macro>
 <xacro:macro name="hokuyo_inertial_params">
@@ -81,13 +84,13 @@
 </xacro:macro>
 <xacro:macro name="left_wheels_collision_geometry">
-  <origin xyz="0 0 -0.0225" rpy="0 0 0" />
+  <origin xyz="0 0 -0.013" rpy="0 0 0" />
   <geometry>
-    <cylinder length="0.045" radius="0.05" />
+    <cylinder length="0.026" radius="0.055" />
   </geometry>
 </xacro:macro>
 <xacro:macro name="right_wheels_collision_geometry">
-  <origin xyz="0 0 0.0225" rpy="0 0 0" />
+  <origin xyz="0 0 0.013" rpy="0 0 0" />
   <geometry>
-    <cylinder length="0.045" radius="0.05" />
+    <cylinder length="0.026" radius="0.055" />
   </geometry>
 </xacro:macro>

File: urdf/unicorn.urdf (robot description, URDF)
Before this commit: robot unicorn, 12 links, 11 joints
Joints:
- joint base_joint: origin xyz=0.0 0.0 -0.05 rpy=0 0 0 -> xyz=0.0 0.0 -0.055 rpy=0 0 0
- joint left_rear_wheel_joint: origin xyz=0 0.1 0 rpy=1.5708 0 0 -> xyz=0 0.148 0 rpy=1.5708 0 0
- joint left_steering_hinge_joint: limit lower=-1.0 upper=1.0 effort=50 velocity=100 -> lower=-1.08 upper=1.08 effort=50 velocity=100; origin xyz=0.325 0.1 0 rpy=0 1.5708 0 -> xyz=0.360 0.151 0 rpy=0 1.5708 0
- joint right_rear_wheel_joint: origin xyz=0 -0.1 0 rpy=1.5708 0 0 -> xyz=0 -0.148 0 rpy=1.5708 0 0
- joint right_steering_hinge_joint: limit lower=-1.0 upper=1.0 effort=50 velocity=100 -> lower=-1.08 upper=1.08 effort=50 velocity=100; origin xyz=0.325 -0.1 0 rpy=0 1.5708 0 -> xyz=0.360 -0.151 0 rpy=0 1.5708 0

Commit message: feat: update vehicle to match Hobao Hyper VS 1/10 specs
- Wheelbase: 325mm -> 360mm
- Front track: 200mm -> 302mm, rear track: 200mm -> 296mm
- Chassis mass: 4.0kg -> 1.7kg, wheel: 0.34kg -> 0.12kg
- Wheel radius: 50mm -> 55mm (110mm diameter)
- Max steering angle: ±1.0 -> ±1.08 rad (62 deg)
- Inertia tensors scaled to match new masses
- Joy teleop: max speed 6 m/s, max steer 1.08 rad
- World STL raised 15cm
- Added TODO.md for remaining work

File: urdf/macros.xacro (robot description, xacro)
@@ -3,26 +3,23 @@
 <!-- inertial parameter macros -->
 <xacro:macro name="chassis_inertial_params">
-  <!-- CoG at ~half wheelbase forward from rear axle (base_link) -->
-  <origin xyz="0.18 0 0" rpy="0 0 0" />
+  <origin xyz="0.1477 0 0" rpy="0 0 0" />
   <mass value="1.70" />
-  <!-- Box approx: 0.56 x 0.302 x 0.06, m=1.7 -->
-  <inertia ixx="0.01343" ixy="0"          ixz="0"
-                          iyy="0.04494"   iyz="0"
-                                           izz="0.05739" />
+  <inertia ixx="0.004509" ixy="0"          ixz="0"
+                          iyy="0.021424"   iyz="0"
+                                           izz="0.024926" />
 </xacro:macro>
 <xacro:macro name="left_wheels_inertial_params">
-  <origin xyz="0 0 -0.013" rpy="0 0 0" />
+  <origin xyz="0 0 -0.0225" rpy="0 0 0" />
   <mass value="0.12" />
-  <!-- Cylinder: r=0.055, h=0.026, m=0.12 -->
-  <inertia ixx="0.0000975" ixy="0"          ixz="0"
-                            iyy="0.0000975" iyz="0"
-                                             izz="0.0001815" />
+  <inertia ixx="0.0000917" ixy="0"          ixz="0"
+                            iyy="0.0000917" iyz="0"
+                                             izz="0.0001452" />
 </xacro:macro>
 <xacro:macro name="right_wheels_inertial_params">
-  <origin xyz="0 0 0.013" rpy="0 0 0" />
+  <origin xyz="0 0 0.0225" rpy="0 0 0" />
   <mass value="0.12" />
-  <inertia ixx="0.0000975" ixy="0"          ixz="0"
-                            iyy="0.0000975" iyz="0"
-                                             izz="0.0001815" />
+  <inertia ixx="0.0000917" ixy="0"          ixz="0"
+                            iyy="0.0000917" iyz="0"
+                                             izz="0.0001452" />
 </xacro:macro>
 <xacro:macro name="steering_hinge_inertial_params">
@@ -36,7 +33,7 @@
   <origin xyz="0 0 0" rpy="0 0 0" />
   <mass value="0.130" />
-  <inertia ixx="4E-06" ixy="0"           ixz="0"
-                            iyy="4E-06"  iyz="0"
-                                              izz="4E-06" />
+  <inertia ixx="2E-06" ixy="0"           ixz="0"
+                            iyy="2E-06"  iyz="0"
+                                              izz="2E-06" />
 </xacro:macro>
 <!-- geometry macros -->
@@ -84,13 +81,13 @@
 </xacro:macro>
 <xacro:macro name="left_wheels_collision_geometry">
-  <origin xyz="0 0 -0.013" rpy="0 0 0" />
+  <origin xyz="0 0 -0.0225" rpy="0 0 0" />
   <geometry>
-    <cylinder length="0.026" radius="0.055" />
+    <cylinder length="0.045" radius="0.055" />
   </geometry>
 </xacro:macro>
 <xacro:macro name="right_wheels_collision_geometry">
-  <origin xyz="0 0 0.013" rpy="0 0 0" />
+  <origin xyz="0 0 0.0225" rpy="0 0 0" />
   <geometry>
-    <cylinder length="0.026" radius="0.055" />
+    <cylinder length="0.045" radius="0.055" />
   </geometry>
 </xacro:macro>

Commit message: fix: adjust vehicle dimensions and track height
- Track width: 302mm -> 255mm (300mm total with 45mm tires)
- Chassis mass: 4.0kg -> 1.7kg, wheel: 0.34kg -> 0.12kg
- Wheel radius: 50mm -> 55mm, CoG adjusted for 360mm wheelbase
- Inertia tensors preserved from original model
- Track STL raised 15.5cm via link pose
- Joy max speed 6 m/s, steering limit 1.08 rad
- Updated TODO with track mesh fix needed

File: urdf/macros.xacro (robot description, xacro)
@@ -3,37 +3,37 @@
 <!-- inertial parameter macros -->
 <xacro:macro name="chassis_inertial_params">
-  <origin xyz="0.1477 0 0" rpy="0 0 0" />
+  <origin xyz="0.18 0 0" rpy="0 0 0" />
   <mass value="1.70" />
-  <inertia ixx="0.004509" ixy="0"          ixz="0"
-                          iyy="0.021424"   iyz="0"
-                                           izz="0.024926" />
+  <inertia ixx="0.010609" ixy="0"          ixz="0"
+                          iyy="0.050409"   iyz="0"
+                                           izz="0.05865" />
 </xacro:macro>
 <xacro:macro name="left_wheels_inertial_params">
   <origin xyz="0 0 -0.0225" rpy="0 0 0" />
   <mass value="0.12" />
-  <inertia ixx="0.0000917" ixy="0"          ixz="0"
-                            iyy="0.0000917" iyz="0"
-                                             izz="0.0001452" />
+  <inertia ixx="0.00026046" ixy="0"          ixz="0"
+                            iyy="0.00026046" iyz="0"
+                                             izz="0.00041226" />
 </xacro:macro>
 <xacro:macro name="right_wheels_inertial_params">
   <origin xyz="0 0 0.0225" rpy="0 0 0" />
   <mass value="0.12" />
-  <inertia ixx="0.0000917" ixy="0"          ixz="0"
-                            iyy="0.0000917" iyz="0"
-                                             izz="0.0001452" />
+  <inertia ixx="0.00026046" ixy="0"          ixz="0"
+                            iyy="0.00026046" iyz="0"
+                                             izz="0.00041226" />
 </xacro:macro>
 <xacro:macro name="steering_hinge_inertial_params">
   <origin xyz="0 0 0" rpy="0 0 0" />
   <mass value="0.05" />
-  <inertia ixx="2E-06" ixy="0"           ixz="0"
-                            iyy="2E-06"  iyz="0"
-                                              izz="2E-06" />
+  <inertia ixx="4E-06" ixy="0"           ixz="0"
+                            iyy="4E-06"  iyz="0"
+                                              izz="4E-06" />
 </xacro:macro>
 <xacro:macro name="hokuyo_inertial_params">
   <origin xyz="0 0 0" rpy="0 0 0" />
   <mass value="0.130" />
-  <inertia ixx="2E-06" ixy="0"           ixz="0"
-                            iyy="2E-06"  iyz="0"
-                                              izz="2E-06" />
+  <inertia ixx="4E-06" ixy="0"           ixz="0"
+                            iyy="4E-06"  iyz="0"
+                                              izz="4E-06" />
 </xacro:macro>
 <!-- geometry macros -->

File: urdf/unicorn.urdf (robot description, URDF)
Before this commit: robot unicorn, 12 links, 11 joints
Joints:
- joint base_joint: origin xyz=0.0 0.0 -0.055 rpy=0 0 0 -> xyz=0.0 0.0 -0.05 rpy=0 0 0
- joint left_rear_wheel_joint: origin xyz=0 0.148 0 rpy=1.5708 0 0 -> xyz=0 0.1275 0 rpy=1.5708 0 0
- joint left_steering_hinge_joint: origin xyz=0.360 0.151 0 rpy=0 1.5708 0 -> xyz=0.360 0.1275 0 rpy=0 1.5708 0
- joint right_rear_wheel_joint: origin xyz=0 -0.148 0 rpy=1.5708 0 0 -> xyz=0 -0.1275 0 rpy=1.5708 0 0
- joint right_steering_hinge_joint: origin xyz=0.360 -0.151 0 rpy=0 1.5708 0 -> xyz=0.360 -0.1275 0 rpy=0 1.5708 0

Commit message: Update chassis mass to 3.655kg for ~4.5kg total vehicle weight
Scale inertia tensor proportionally (x2.15) to match new mass.

File: urdf/macros.xacro (robot description, xacro)
@@ -4,8 +4,8 @@
 <xacro:macro name="chassis_inertial_params">
   <origin xyz="0.18 0 0" rpy="0 0 0" />
-  <mass value="1.70" />
-  <inertia ixx="0.010609" ixy="0"          ixz="0"
-                          iyy="0.050409"   iyz="0"
-                                           izz="0.05865" />
+  <mass value="3.655" />
+  <inertia ixx="0.022809" ixy="0"          ixz="0"
+                          iyy="0.108379"   iyz="0"
+                                           izz="0.126098" />
 </xacro:macro>
 <xacro:macro name="left_wheels_inertial_params">

Commit message: feat: change  package name

File: urdf/macros.xacro (robot description, xacro)
@@ -41,5 +41,5 @@
   <origin xyz="0 0 0" rpy="0 0 0" />
   <geometry>
-    <mesh filename="package://unicorn_model/meshes/chassis.STL"/>
+    <mesh filename="package://roboracer_gazebo/meshes/chassis.STL"/>
   </geometry>
 </xacro:macro>
@@ -47,5 +47,5 @@
   <origin xyz="0 0 0" rpy="0 0 0" />
   <geometry>
-    <mesh filename="package://unicorn_model/meshes/left_rear_wheel.STL"/>
+    <mesh filename="package://roboracer_gazebo/meshes/left_rear_wheel.STL"/>
   </geometry>
 </xacro:macro>
@@ -53,5 +53,5 @@
   <origin xyz="0 0 0" rpy="0 0 0" />
   <geometry>
-    <mesh filename="package://unicorn_model/meshes/right_rear_wheel.STL"/>
+    <mesh filename="package://roboracer_gazebo/meshes/right_rear_wheel.STL"/>
   </geometry>
 </xacro:macro>
@@ -59,5 +59,5 @@
   <origin xyz="0 0 0" rpy="0 0 0" />
   <geometry>
-    <mesh filename="package://unicorn_model/meshes/left_front_wheel.STL"/>
+    <mesh filename="package://roboracer_gazebo/meshes/left_front_wheel.STL"/>
   </geometry>
 </xacro:macro>
@@ -65,5 +65,5 @@
   <origin xyz="0 0 0" rpy="0 0 0" />
   <geometry>
-    <mesh filename="package://unicorn_model/meshes/right_front_wheel.STL"/>
+    <mesh filename="package://roboracer_gazebo/meshes/right_front_wheel.STL"/>
   </geometry>
 </xacro:macro>
@@ -71,5 +71,5 @@
   <origin xyz="0 0 0" rpy="0 0 0" />
   <geometry>
-    <mesh filename="package://unicorn_model/meshes/left_steering_hinge.STL"/>
+    <mesh filename="package://roboracer_gazebo/meshes/left_steering_hinge.STL"/>
   </geometry>
 </xacro:macro>
@@ -77,5 +77,5 @@
   <origin xyz="0 0 0" rpy="0 0 0" />
   <geometry>
-    <mesh filename="package://unicorn_model/meshes/right_steering_hinge.STL"/>
+    <mesh filename="package://roboracer_gazebo/meshes/right_steering_hinge.STL"/>
   </geometry>
 </xacro:macro>
